Commit message: Reworked some KDL FK computation.

File: data/planar_2dof/planar_2dof.urdf (robot description, URDF)
Before this commit: robot 2dof, 3 links, 2 joints
Links:
- added link tool
Joints:
- added joint ee: type fixed, parent link2, child tool, origin xyz=0.5 0 0 rpy=0 0 0, axis 0 0 1, limit lower=-6.28318 upper=6.28318 effort=30 velocity=1.0
- joint joint1: limit (none) -> lower=-1.570795 upper=1.570795 effort=30 velocity=1.0; type continuous -> revolute
- joint joint2: limit (none) -> lower=-1.570795 upper=1.570795 effort=30 velocity=1.0; type continuous -> revolute

Commit message: Investigating KDL-FCL screwups

File: data/planar_2dof/planar_2dof.urdf (robot description, URDF)
Before this commit: robot 2dof, 4 links, 3 joints
Joints:
- joint joint1: limit lower=-1.570795 upper=1.570795 effort=30 velocity=1.0 -> lower=-3.14158 upper=3.14158 effort=30 velocity=1.0
- joint joint2: limit lower=-1.570795 upper=1.570795 effort=30 velocity=1.0 -> lower=-3.14158 upper=3.14158 effort=30 velocity=1.0

Commit message: Finished implementint RRTConnect for Planar2DOF

File: data/planar_2dof/planar_2dof.urdf (robot description, URDF)
Before this commit: robot 2dof, 4 links, 3 joints
Joints:
- joint joint1: limit lower=-3.14158 upper=3.14158 effort=30 velocity=1.0 -> lower=-2.9 upper=2.9 effort=30 velocity=1.0
- joint joint2: limit lower=-3.14158 upper=3.14158 effort=30 velocity=1.0 -> lower=-2.9 upper=2.9 effort=30 velocity=1.0

Commit message: Obstacles are now read from yaml file, RRTConnect is running flawlessly

File: data/planar_2dof/planar_2dof.urdf (robot description, URDF)
Before this commit: robot 2dof, 4 links, 3 joints
Joints:
- joint joint1: limit lower=-2.9 upper=2.9 effort=30 velocity=1.0 -> lower=-2.6 upper=2.6 effort=30 velocity=1.0
- joint joint2: limit lower=-2.9 upper=2.9 effort=30 velocity=1.0 -> lower=-2.6 upper=2.6 effort=30 velocity=1.0

Commit message: RGBMTStar buggs fixed. Work well for tested scenarios.

File: data/planar_2dof/planar_2dof.urdf (robot description, URDF)
Before this commit: robot 2dof, 4 links, 3 joints
Links:
- link link2: geometry visual box size=1 0.05 0.05
Joints:
- joint joint1: limit lower=-2.6 upper=2.6 effort=30 velocity=1.0 -> lower=-3.14159 upper=3.14159 effort=30 velocity=1.0
- joint joint2: limit lower=-2.6 upper=2.6 effort=30 velocity=1.0 -> lower=-3.14159 upper=3.14159 effort=30 velocity=1.0

Commit message: Cannot find bug in connectGenSpine

File: data/planar_2dof/planar_2dof.urdf (robot description, URDF)
Before this commit: robot 2dof, 4 links, 3 joints
Joints:
- joint joint1: limit lower=-3.14159 upper=3.14159 effort=30 velocity=1.0 -> lower=-3 upper=3 effort=30 velocity=1.0
- joint joint2: limit lower=-3.14159 upper=3.14159 effort=30 velocity=1.0 -> lower=-3 upper=3 effort=30 velocity=1.0

Commit message: RGBMTStar is now working flawlessly

File: data/planar_2dof/planar_2dof.urdf (robot description, URDF)
Before this commit: robot 2dof, 4 links, 3 joints
Joints:
- joint ee: origin xyz=0.5 0 0 rpy=0 0 0 -> xyz=1 0 0 rpy=0 0 0
- joint joint1: limit lower=-3 upper=3 effort=30 velocity=1.0 -> lower=-3.14159 upper=3.14159 effort=30 velocity=1.0
- joint joint2: limit lower=-3 upper=3 effort=30 velocity=1.0 -> lower=-3.14159 upper=3.14159 effort=30 velocity=1.0
